File: hawb-board.sch (EAGLE design)
At the start: 85 parts, among them IC1 3.3V SR05S3V3, IC2 5V SR05S05, IC3 OPAMP-DUALU, IC4 OPAMP-DUALU, M2 HX1, Q1 MOSFET-NCHANNELFDD8580, Q2 MOSFET-NCHANNELFDD8580, Q3 N-FET, Q4 N-FET, Q5 N-FET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

Commit message: Added some decoupling caps, bom
Parts:
- added C11, C7: 0.1uF, rcl:C-EUC0603
- C5: device sparkfun:CAP0402-CAP -> SparkFun-Capacitors:CAP0603-CAP
Connections:
- net 5V: now also C11.1, C7.1
- net GND: now also C11.2, C7.2
Changed lines of the file:
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@@
 <part name="U$5" library="sparkfun" deviceset="5V" device=""/>
 <part name="GND19" library="sparkfun" deviceset="GND" device=""/>
-<part name="C5" library="sparkfun" deviceset="CAP" device="0402-CAP" value="1nF"/>
+<part name="C5" library="SparkFun-Capacitors" deviceset="CAP" device="0603-CAP" value="1nF"/>
 <part name="IC4" library="sparkfun" deviceset="OPAMP-DUAL" device="U"/>
 <part name="U$11" library="sparkfun" deviceset="5V" device=""/>
@@
 <part name="T6" library="SparkFun-Connectors" deviceset="M01" device="PTH"/>
 <part name="T7" library="SparkFun-Connectors" deviceset="M01" device="PTH"/>
+<part name="C7" library="rcl" deviceset="C-EU" device="C0603" value="0.1uF"/>
+<part name="U$15" library="sparkfun" deviceset="5V" device=""/>
+<part name="GND33" library="sparkfun" deviceset="GND" device=""/>
+<part name="C11" library="rcl" deviceset="C-EU" device="C0603" value="0.1uF"/>
+<part name="U$16" library="sparkfun" deviceset="5V" device=""/>
+<part name="GND34" library="sparkfun" deviceset="GND" device=""/>
 </parts>
 <sheets>
@@
 <instance part="R11" gate="G$1" x="-152.4" y="88.9" rot="R90"/>
 <instance part="R12" gate="G$1" x="-152.4" y="73.66" rot="R90"/>
-<instance part="U$5" gate="G$1" x="-137.16" y="114.3"/>
+<instance part="U$5" gate="G$1" x="-137.16" y="116.84"/>
 <instance part="GND19" gate="1" x="-137.16" y="91.44"/>
 <instance part="C5" gate="G$1" x="-119.38" y="104.14" rot="R270"/>
@@
 <instance part="T6" gate="G$1" x="-68.58" y="10.16" rot="R90"/>
 <instance part="T7" gate="G$1" x="45.72" y="109.22" rot="R270"/>
+<instance part="C7" gate="G$1" x="-137.16" y="73.66"/>
+<instance part="U$15" gate="G$1" x="-137.16" y="78.74"/>
+<instance part="GND33" gate="1" x="-137.16" y="63.5"/>
+<instance part="C11" gate="G$1" x="-137.16" y="0"/>
+<instance part="U$16" gate="G$1" x="-137.16" y="5.08"/>
+<instance part="GND34" gate="1" x="-137.16" y="-10.16"/>
 </instances>
 <busses>
@@
 <wire x1="137.16" y1="96.52" x2="137.16" y2="93.98" width="0.1524" layer="91"/>
 </segment>
+<segment>
+<pinref part="C7" gate="G$1" pin="2"/>
+<pinref part="GND33" gate="1" pin="GND"/>
+<wire x1="-137.16" y1="68.58" x2="-137.16" y2="66.04" width="0.1524" layer="91"/>
+</segment>
+<segment>
+<pinref part="C11" gate="G$1" pin="2"/>
+<pinref part="GND34" gate="1" pin="GND"/>
+<wire x1="-137.16" y1="-5.08" x2="-137.16" y2="-7.62" width="0.1524" layer="91"/>
+</segment>
 </net>
 <net name="5V" class="0">
@@
 <pinref part="U$5" gate="G$1" pin="5V"/>
 <pinref part="IC3" gate="A" pin="V+"/>
-<wire x1="-137.16" y1="114.3" x2="-137.16" y2="111.76" width="0.1524" layer="91"/>
+<wire x1="-137.16" y1="116.84" x2="-137.16" y2="111.76" width="0.1524" layer="91"/>
 </segment>
 <segment>
@@
 <wire x1="-101.6" y1="38.1" x2="-101.6" y2="35.56" width="0.1524" layer="91"/>
 </segment>
-</net>
+<segment>
+<pinref part="U$15" gate="G$1" pin="5V"/>
+<pinref part="C7" gate="G$1" pin="1"/>
+<wire x1="-137.16" y1="78.74" x2="-137.16" y2="76.2" width="0.1524" layer="91"/>
+</segment>
+<segment>
+<pinref part="U$16" gate="G$1" pin="5V"/>
+<pinref part="C11" gate="G$1" pin="1"/>
+<wire x1="-137.16" y1="5.08" x2="-137.16" y2="2.54" width="0.1524" layer="91"/>
+</segment>
+</net>
